Commit message: feat: M3 全链路验收——CMU 导航栈驱动 Go2W 在 warehouse 自主导航
验收证据：waypoint (2.5,0) -> SLAM 轨迹 0.76->2.46m 收敛到目标；地面真值
(3.19,-0.75) 与 SLAM+原点偏移交叉验证一致；全程站高 0.37m；静止漂移 5cm/20s；
截图存档 logs/nav_shots5。

新增：warehouse_nav.py（RTX 雷达 + 物理正确 IMU + /clock + cmd_vel 差速执行，
全 sim-time）；pc2_to_livox.py（PointCloud2->CustomMsg，回溯帧戳）；
run_navstack.sh（容器内编排）；patch_navstack.sh（对干净导航栈克隆一键应用
全部集成修改，refs/ 不入库）；Livox_Mid360_approx 雷达配置生成器 + USD。

深坑（README 16-22 全记录）：Kit 时间线倍速（render_interval 必须=1 且 dt 一致）；
雷达帧戳来自未来（回溯修复，sync 警告 225->1）；isaaclab Imu gravity_bias 斜装
错误（按姿态投影）；100Hz 物理下腿 PD 需 100/5；DDS 域隔离(42)；ldconfig；
set -u 吃 ROS setup。轮碰撞体网格->圆柱（拖滞修复，自检 PASS）。

未竟：D435 深度图输出、PiPER ROS2 控制接口（M2 收尾）；y 向 SLAM 漂移 ~0.2m/3m
待调；tare_planner 未编译（探索模式暂缺）。

File: assets/urdf/go2w_sensored.urdf (robot description, URDF)
Before this commit: robot go2w_sensored, 48 links, 47 joints
Links:
- link FL_foot: geometry collision cylinder length=0.052 radius=0.086; visual mesh filename=../unitree_ros/robots/go2w_description/dae/left_wheel.dae
- link FR_foot: geometry collision cylinder length=0.052 radius=0.086; visual mesh filename=../unitree_ros/robots/go2w_description/dae/right_wheel.dae
- link RL_foot: geometry collision cylinder length=0.052 radius=0.086; visual mesh filename=../unitree_ros/robots/go2w_description/dae/left_wheel.dae
- link RR_foot: geometry collision cylinder length=0.052 radius=0.086; visual mesh filename=../unitree_ros/robots/go2w_description/dae/right_wheel.dae

Commit message: fix(urdf): nuc_weight 0.5kg 占位 -> 1.8kg 实测值——载荷保真修复(CEO 载荷轮指示)
依据:vx-audit 实物 ~1.8kg;runbook payload-fidelity 注。重核算:审计口径载荷
(PiPER 4.660+NUC 1.8)=6.460kg≈审计 ~6.5(原占位仅 5.16);背部总挂 7.463;全挂载 7.800。
惯量按盒体公式(0.11x0.10x0.05)随质量重算(ixx 0.001875/iyy 0.00219/izz 0.003315)。
裸机变体 make_bare_urdf.py 再生成(nuc 不在裸机,字节级不变,确认剥离正确)。
训练载荷中心(plan-a 5-8kg add)/部署 URDF/实物三者对齐。sim-plan 载荷表同步。

File: assets/urdf/go2w_sensored.urdf (robot description, URDF)
Before this commit: robot go2w_sensored, 48 links, 47 joints
Links:
- link nuc_weight: mass 0.5 -> 1.8

Commit message: enlarge Mid-360 collision envelope

File: assets/urdf/go2w_sensored.urdf (robot description, URDF)
Before this commit: robot go2w_sensored, 48 links, 47 joints
Links:
- link mid360_link: geometry collision cylinder length=0.075 radius=0.042; visual mesh filename=../sensor_meshes/mid360.stl scale=0.001 0.001 0.001

Commit message: Calibrate PiPER mount transform

File: assets/urdf/go2w_sensored.urdf (robot description, URDF)
Before this commit: robot go2w_sensored, 48 links, 47 joints
Joints:
- joint piper_mount_joint: origin xyz=0.06 0.0 0.067 rpy=0 0 0 -> xyz=0.128526599 0.0 0.081794287 rpy=0 0 0

Commit message: Move the Mid-360 to its measured pose and model its bracket
mid360_joint 0.27/0/0.10 -> 0.33/0/0.14 (operator-approved against a
photograph of the real head), plus a new mid360_bracket_link box for the
70x70x83 mm mounting post, which had no collision representation at all.

THIS CHANGES NOTHING AT RUNTIME, and the comments in the file say so.
Z-Mobile-manip's PinocchioSelfCollisionChecker reduces the model to the six
active PiPER joints, so every geometry fixed to `base` -- including these --
is dropped before a single collision pair is built.  That is why e4be019
'enlarge Mid-360 collision envelope' (this repo) had zero effect on the
planner, and why a8ecd46 could then shrink the *enforced* capsule in
Z-Mobile-manip/configs/piper_collision_capsules.json from 0.042 to 0.0325
without anyone noticing.

This edit exists for MuJoCo/RViz truth and as the source of truth for
Z-Mobile-manip tests/test_lidar_keepout.py, which recomputes the enforced
capsules from this file and fails if the two ever drift apart again.

File: assets/urdf/go2w_sensored.urdf (robot description, URDF)
Before this commit: robot go2w_sensored, 48 links, 47 joints
Links:
- added link mid360_bracket_link; collision box size=0.07 0.07 0.083
Joints:
- added joint mid360_bracket_joint: type fixed, parent base, child mid360_bracket_link, origin xyz=0.317174 0.0 0.0985 rpy=0 0 0
- joint mid360_joint: origin xyz=0.27 0.0 0.1 rpy=0 0.3490658503988659 0 -> xyz=0.33 0.0 0.14 rpy=0 0.3490658503988659 0
